Commit message: 增加了机械臂底座

File: src/wheel_dual_arm_robot/urdf/wheel_dual_arm_robot.urdf (robot description, URDF)
Before this commit: robot wheel_dual_arm_robot, 5 links, 4 joints
Links:
- link b-l1: mass 3.3026 -> 3.30257766952345
- link b-l2: mass 4.3356 -> 4.33563046644472
- link b-l3: mass 5.2703 -> 5.27028256939189
- link base_arm_link: mass 0.00425983303776923 -> 1.88365700165481
- link base_link: mass 6.8621 -> 6.86209526220681

Commit message: 增加机械臂j1关节，正常旋转

File: src/wheel_dual_arm_robot/urdf/wheel_dual_arm_robot.urdf (robot description, URDF)
Before this commit: robot wheel_dual_arm_robot, 5 links, 4 joints
Links:
- removed link b-l1
- removed link b-l2
- removed link b-l3
- removed link base_arm_link
- added link arm_base_link, mass 1.8837; collision mesh filename=package://wheel_dual_arm_robot/meshes/arm_base_link.STL; visual mesh filename=package://wheel_dual_arm_robot/meshes/arm_base_link.STL
- added link b1, mass 3.30257766952345; collision mesh filename=package://wheel_dual_arm_robot/meshes/b1.STL; visual mesh filename=package://wheel_dual_arm_robot/meshes/b1.STL
- added link b2, mass 4.33563046644472; collision mesh filename=package://wheel_dual_arm_robot/meshes/b2.STL; visual mesh filename=package://wheel_dual_arm_robot/meshes/b2.STL
- added link b3, mass 5.2703; collision mesh filename=package://wheel_dual_arm_robot/meshes/b3.STL; visual mesh filename=package://wheel_dual_arm_robot/meshes/b3.STL
- added link l1, mass 0.53062; collision mesh filename=package://wheel_dual_arm_robot/meshes/l1.STL; visual mesh filename=package://wheel_dual_arm_robot/meshes/l1.STL
- added link r1, mass 0.53062; collision mesh filename=package://wheel_dual_arm_robot/meshes/r1.STL; visual mesh filename=package://wheel_dual_arm_robot/meshes/r1.STL
- link base_link: mass 6.86209526220681 -> 6.86209515901701
Joints:
- removed joint base_arm-j0
- added joint body_to_arm: type fixed, parent b3, child arm_base_link, origin xyz=0.454 0 0 rpy=1.5708 0 1.5708, axis 0 0 0
- added joint l-j1: type revolute, parent arm_base_link, child l1, origin xyz=0 0.225 0 rpy=-1.5708 1.5708 0, axis 0 0 1, limit lower=-6.2832 upper=6.2832 effort=0 velocity=0
- added joint r-j1: type revolute, parent arm_base_link, child r1, origin xyz=0 -0.225 0 rpy=1.5708 -1.5708 0, axis 0 0 1, limit lower=-6.2832 upper=6.2832 effort=0 velocity=0
- joint b-j1: child b-l1 -> b1; limit lower=-3.1416 upper=3.1416 effort=0 velocity=0 -> lower=-6.2832 upper=6.2832 effort=0 velocity=0
- joint b-j2: child b-l2 -> b2; limit lower=-3.1416 upper=3.1416 effort=0 velocity=0 -> lower=-6.2832 upper=6.2832 effort=0 velocity=0; parent b-l1 -> b1
- joint b-j3: child b-l3 -> b3; limit lower=-3.1416 upper=3.1416 effort=0 velocity=0 -> lower=-6.2832 upper=6.2832 effort=0 velocity=0; parent b-l2 -> b2
